File: PCB/ZPansion/ZPansion.kicad_sch (KiCad schematic)
At the start: 20 parts, among them M1 D24V5F12, M2 TMCSILENTSTEPSTICK, M3 TMCSILENTSTEPSTICK, M4 TMCSILENTSTEPSTICK, T1 PRPC005DAAN-RC, T2 0395121002, T3 0395121004, T4 0395121004, T5 0395121004

Commit message: PCB Done
 Finished PCB design and route. Schematic tweaked along the way, termination resistors added to SPI just in case.
Parts:
- added C9: UCM1C470MCL1GS, AVR-KiCAD-Lib-Capacitors:UCM1C470MCL1GS, symbol AVR-KiCAD-Lib-Capacitors:UCM1C470MCL1GS
- added H1, H2, H3, H4: M3_Plated_Hole, AVR-KiCAD-Lib-Holes_Fasteners:M3_HOLE, symbol AVR-KiCAD-Lib-Holes_Fasteners:M3_Plated_Hole
- added R2: RC0402FR-071KL, AVR-KiCAD-Lib-Resistors:R0402, symbol AVR-KiCAD-Lib-Resistors:RC0402FR-071KL
- added R3, R4, R5: RC0402FR-0722RL, AVR-KiCAD-Lib-Resistors:R0402, symbol AVR-KiCAD-Lib-Resistors:RC0402FR-0722RL
- added R6, R7, R8: RC0402FR-0710KL, AVR-KiCAD-Lib-Resistors:R0402, symbol AVR-KiCAD-Lib-Resistors:RC0402FR-0710KL
- added T10, T11, T6, T7, T8, T9: 0705430002, AVR-KiCAD-Lib-Connectors:Shrouded_Pin_Header_Straight_1x03_Pitch2.54mm, symbol AVR-KiCAD-Lib-Connectors:0705430002
- T1: footprint Pin_Headers:Pin_Header_Straight_2x05_Pitch2.54mm -> Connector_PinHeader_2.54mm:PinHeader_2x05_P2.54mm_Vertical
Connections:
- net +3V3: now also C9.1, R2.2, R6.2, R7.2, R8.2, T10.2, T11.2, T6.2, T7.2, T8.2, T9.2
- net ENABLE: now also SP1.9 (4/A6)
- net GND: now also C9.2, T10.3, T11.3, T6.3, T7.3, T8.3, T9.3
- net MASTER_DIR: now also T1.5; no longer T1.7
- net MASTER_STEP: now also T1.7; no longer T1.5
- net SPI_CS0: now also R8.1
- net SPI_CS1: now also R6.1
- net SPI_CS2: now also R7.1
- net SPI_SCK: now also R3.1; no longer M2.7 (SPI_SDI), M3.7 (SPI_SDI), M4.7 (SPI_SDI)
- net SPI_SDI: now also R5.1; no longer M2.6 (SPI_SCK), M3.6 (SPI_SCK), M4.6 (SPI_SCK)
- net SPI_SDO: now also R4.1; no longer M2.4 (SPI_SDO), M3.4 (SPI_SDO), M4.4 (SPI_SDO)
- net SYS_RESET: now also R2.1
- net UART_RX: now also T1.3; no longer T1.1
- net UART_TX: now also T1.1; no longer T1.3
- net at SP1.21 (A0): now also T6.1
- net at SP1.22 (A1): now also T7.1
- net at SP1.23 (A2): now also T8.1
- net at SP1.24 (A3): now also T9.1
- net at SP1.25 (A4): now also T10.1
- net at SP1.26 (A5): now also T11.1
- new net: M2.4 (SPI_SDO), M3.4 (SPI_SDO), M4.4 (SPI_SDO), R4.2
- new net: M2.6 (SPI_SCK), M3.6 (SPI_SCK), M4.6 (SPI_SCK), R5.2
- new net: M2.7 (SPI_SDI), M3.7 (SPI_SDI), M4.7 (SPI_SDI), R3.2
- new net GNDREF: H1.1, H2.1, H3.1, H4.1
Other:
- moved on the sheet: C1, C2, C3, C4, C5, C6, C7, C8, D1, M1, M2, M3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
